Commit message: Adding new ROS2 workspace files

File: src/moveit_config/config/my_robot.ros2_control.xacro (robot description, xacro)
@@ -8,4 +8,5 @@
                 <plugin>mock_components/GenericSystem</plugin>
             </hardware>
+<<<<<<< HEAD
             <joint name="base_link_Slider-13">
                 <command_interface name="position"/>
@@ -40,4 +41,38 @@
                 <state_interface name="position">
                   <param name="initial_value">${initial_positions['MOTOR_Revolute-17']}</param>
+=======
+            <joint name="BASE_Slider-1">
+                <command_interface name="position"/>
+                <state_interface name="position">
+                  <param name="initial_value">${initial_positions['BASE_Slider-1']}</param>
+                </state_interface>
+                <state_interface name="velocity"/>
+            </joint>
+            <joint name="LINK1_Revolute-2">
+                <command_interface name="position"/>
+                <state_interface name="position">
+                  <param name="initial_value">${initial_positions['LINK1_Revolute-2']}</param>
+                </state_interface>
+                <state_interface name="velocity"/>
+            </joint>
+            <joint name="LINK2_Revolute-3">
+                <command_interface name="position"/>
+                <state_interface name="position">
+                  <param name="initial_value">${initial_positions['LINK2_Revolute-3']}</param>
+                </state_interface>
+                <state_interface name="velocity"/>
+            </joint>
+            <joint name="LINK3_Revolute-4">
+                <command_interface name="position"/>
+                <state_interface name="position">
+                  <param name="initial_value">${initial_positions['LINK3_Revolute-4']}</param>
+                </state_interface>
+                <state_interface name="velocity"/>
+            </joint>
+            <joint name="LINK4_Revolute-5">
+                <command_interface name="position"/>
+                <state_interface name="position">
+                  <param name="initial_value">${initial_positions['LINK4_Revolute-5']}</param>
+>>>>>>> 1a366d7 (Adding new ROS2 workspace files)
                 </state_interface>
                 <state_interface name="velocity"/>

File: src/moveit_config/config/my_robot.urdf.xacro (robot description, xacro)
@@ -3,5 +3,9 @@
     <xacro:arg name="initial_positions_file" default="initial_positions.yaml" />
     <!-- Import my_robot urdf file -->
+<<<<<<< HEAD
     <xacro:include filename="$(find my_robot_description)/urdf/my_robot.urdf.xacro" />
+=======
+    <xacro:include filename="$(find my_robot_description)/urdf/my_robot_processed.urdf" />
+>>>>>>> 1a366d7 (Adding new ROS2 workspace files)
     <!-- Import control_xacro -->
     <xacro:include filename="my_robot.ros2_control.xacro" />
